File: pcb/Matrix.kicad_sch (KiCad schematic)
At the start: 114 parts

Commit message: 🛠️ Remove unwanted layouts
Parts:
- removed D42, D44: DIODE, Diode_THT:D_DO-35_SOD27_P7.62mm_Horizontal, symbol Device:D_Small_Filled
- removed S53, S66: SWITCH_2PIN, ElsassKabel:SW_Cherry_MX_PCB_6.25u, symbol Switch:SW_Push
- removed S54, S59, S61: SWITCH_2PIN, ElsassKabel:SW_Cherry_MX_PCB_1.00u, symbol Switch:SW_Push
- removed S55, S57, S58, S63, S64, S65: SWITCH_2PIN, ElsassKabel:SW_Cherry_MX_PCB_1.25u, symbol Switch:SW_Push
- removed S56: SWITCH_2PIN, ElsassKabel:SW_Cherry_MX_PCB_7.00u, symbol Switch:SW_Push
- removed S60: SWITCH_2PIN, ElsassKabel:SW_Cherry_MX_PCB_2.25u, symbol Switch:SW_Push
- removed S62: SWITCH_2PIN, ElsassKabel:SW_Cherry_MX_PCB_2.75u, symbol Switch:SW_Push
